File: PCBs_OpA/HPF.sch (KiCad schematic (older format))
At the start: 9 parts, among them J5 MEASURE, J7 MEASURE

Commit message: operational amplifier Direct detection receiver
Parts:
- removed L19: 1uH, Choke_Axial_ThroughHole:Choke_Horizontal_RM10mm, symbol L_Small
- added C21: 1nF, LCSDR:C_1206_0603, symbol C_Small
- C45: value 330pF -> 360pF
- C47: value 220pF -> 360pF
- C49: value 330pF -> 1nF
- L13: footprint Choke_Axial_ThroughHole:Choke_Horizontal_RM10mm -> Choke_Toroid_ThroughHole:Choke_Toroid_6,5x13mm_Vertical
- L15: footprint Resistors_THT:R_Axial_DIN0309_L9.0mm_D3.2mm_P2.54mm_Vertical -> Choke_Toroid_ThroughHole:Choke_Toroid_6,5x13mm_Vertical
- L17: value 680nH -> 1uH; footprint Choke_Axial_ThroughHole:Choke_Horizontal_RM10mm -> Choke_Toroid_ThroughHole:Choke_Toroid_6,5x13mm_Vertical
Connections:
- net RF_IN: now also C21.1; no longer C45.1, L13.1
- new net: C21.2, C45.1, L13.1
Other:
- moved on the sheet: J5
Changed lines of the file:
@@
 P 3700 2200
 F 0 "C45" V 3950 2150 50  0000 L CNN
-F 1 "330pF" V 3850 2050 50  0000 L CNN
+F 1 "360pF" V 3850 2050 50  0000 L CNN
 F 2 "LCSDR:C_1206_0603" H 3700 2200 50  0001 C CNN
 F 3 "" H 3700 2200 50  0001 C CNN
@@
 P 4550 2200
 F 0 "C47" V 4800 2150 50  0000 L CNN
-F 1 "220pF" V 4700 2050 50  0000 L CNN
+F 1 "360pF" V 4700 2050 50  0000 L CNN
 F 2 "LCSDR:C_1206_0603" H 4550 2200 50  0001 C CNN
 F 3 "" H 4550 2200 50  0001 C CNN
@@
 P 5300 2200
 F 0 "C49" V 5550 2150 50  0000 L CNN
-F 1 "330pF" V 5450 2050 50  0000 L CNN
+F 1 "1nF" V 5450 2050 50  0000 L CNN
 F 2 "LCSDR:C_1206_0603" H 5300 2200 50  0001 C CNN
 F 3 "" H 5300 2200 50  0001 C CNN
@@
 P 4950 2400
 F 0 "L17" H 4980 2440 50  0000 L CNN
-F 1 "680nH" H 4980 2360 50  0000 L CNN
-F 2 "Choke_Axial_ThroughHole:Choke_Horizontal_RM10mm" H 4950 2400 50  0001 C CNN
+F 1 "1uH" H 4980 2360 50  0000 L CNN
+F 2 "Choke_Toroid_ThroughHole:Choke_Toroid_6,5x13mm_Vertical" H 4950 2400 50  0001 C CNN
 F 3 "" H 4950 2400 50  0001 C CNN
 	1    4950 2400
-	1    0    0    -1
-$EndComp
-$Comp
-L L_Small L19
-U 1 1 630A370D
-P 5650 2400
-F 0 "L19" H 5680 2440 50  0000 L CNN
-F 1 "1uH" H 5680 2360 50  0000 L CNN
-F 2 "Choke_Axial_ThroughHole:Choke_Horizontal_RM10mm" H 5650 2400 50  0001 C CNN
-F 3 "" H 5650 2400 50  0001 C CNN
-	1    5650 2400
 	1    0    0    -1
 $EndComp
@@
 F 0 "L15" H 4180 2440 50  0000 L CNN
 F 1 "680nH" H 4180 2360 50  0000 L CNN
-F 2 "Resistors_THT:R_Axial_DIN0309_L9.0mm_D3.2mm_P2.54mm_Vertical" H 4150 2400 50  0001 C CNN
+F 2 "Choke_Toroid_ThroughHole:Choke_Toroid_6,5x13mm_Vertical" H 4150 2400 50  0001 C CNN
 F 3 "" H 4150 2400 50  0001 C CNN
 	1    4150 2400
@@
 F 0 "L13" H 3380 2440 50  0000 L CNN
 F 1 "1uH" H 3380 2360 50  0000 L CNN
-F 2 "Choke_Axial_ThroughHole:Choke_Horizontal_RM10mm" H 3350 2400 50  0001 C CNN
+F 2 "Choke_Toroid_ThroughHole:Choke_Toroid_6,5x13mm_Vertical" H 3350 2400 50  0001 C CNN
 F 3 "" H 3350 2400 50  0001 C CNN
 	1    3350 2400
@@
 $Comp
 L GND #PWR0102
-U 1 1 630A3912
-P 5650 2600
-F 0 "#PWR0102" H 5650 2350 50  0001 C CNN
-F 1 "GND" H 5650 2450 50  0000 C CNN
-F 2 "" H 5650 2600 50  0001 C CNN
-F 3 "" H 5650 2600 50  0001 C CNN
-	1    5650 2600
-	1    0    0    -1
-$EndComp
-$Comp
-L GND #PWR0103
 U 1 1 630A3972
 P 4950 2600
-F 0 "#PWR0103" H 4950 2350 50  0001 C CNN
+F 0 "#PWR0102" H 4950 2350 50  0001 C CNN
 F 1 "GND" H 4950 2450 50  0000 C CNN
 F 2 "" H 4950 2600 50  0001 C CNN
@@
 $EndComp
 $Comp
-L GND #PWR0104
+L GND #PWR0103
 U 1 1 630A39B4
 P 4150 2600
-F 0 "#PWR0104" H 4150 2350 50  0001 C CNN
+F 0 "#PWR0103" H 4150 2350 50  0001 C CNN
 F 1 "GND" H 4150 2450 50  0000 C CNN
 F 2 "" H 4150 2600 50  0001 C CNN
@@
 $EndComp
 $Comp
-L GND #PWR0105
+L GND #PWR0104
 U 1 1 630A39EF
 P 3350 2600
-F 0 "#PWR0105" H 3350 2350 50  0001 C CNN
+F 0 "#PWR0104" H 3350 2350 50  0001 C CNN
 F 1 "GND" H 3350 2450 50  0000 C CNN
 F 2 "" H 3350 2600 50  0001 C CNN
@@
 	5400 2200 6400 2200
 Wire Wire Line
-	5650 2200 5650 2300
-Wire Wire Line
 	3800 2200 4450 2200
 Wire Wire Line
@@
 Connection ~ 4150 2200
 Wire Wire Line
-	2500 2200 3600 2200
-Wire Wire Line
 	3350 2200 3350 2300
-Connection ~ 5650 2200
 Connection ~ 3350 2200
-Wire Wire Line
-	5650 2500 5650 2600
 Wire Wire Line
 	4950 2500 4950 2600
@@
 $EndComp
 $Comp
-L GND #PWR0106
+L GND #PWR0105
 U 1 1 630C7FC1
 P 6250 2750
-F 0 "#PWR0106" H 6250 2500 50  0001 C CNN
+F 0 "#PWR0105" H 6250 2500 50  0001 C CNN
 F 1 "GND" H 6250 2600 50  0001 C CNN
 F 2 "" H 6250 2750 50  0001 C CNN
@@
 L Conn_Coaxial J5
 U 1 1 630C80F5
-P 2850 2500
-F 0 "J5" H 2860 2620 50  0000 C CNN
-F 1 "MEASURE" H 3150 2500 50  0000 C CNN
-F 2 "LCSDR:U.FL_Molex_MCRF_73412-0110_Vertical" H 2850 2500 50  0001 C CNN
-F 3 "" H 2850 2500 50  0001 C CNN
-	1    2850 2500
+P 2300 2500
+F 0 "J5" H 2310 2620 50  0000 C CNN
+F 1 "MEASURE" H 2600 2500 50  0000 C CNN
+F 2 "LCSDR:U.FL_Molex_MCRF_73412-0110_Vertical" H 2300 2500 50  0001 C CNN
+F 3 "" H 2300 2500 50  0001 C CNN
+	1    2300 2500
 	-1   0    0    -1
 $EndComp
 $Comp
-L GND #PWR0107
+L GND #PWR0106
 U 1 1 630C80FB
-P 2850 2750
-F 0 "#PWR0107" H 2850 2500 50  0001 C CNN
-F 1 "GND" H 2850 2600 50  0001 C CNN
-F 2 "" H 2850 2750 50  0001 C CNN
-F 3 "" H 2850 2750 50  0001 C CNN
-	1    2850 2750
+P 2300 2750
+F 0 "#PWR0106" H 2300 2500 50  0001 C CNN
+F 1 "GND" H 2300 2600 50  0001 C CNN
+F 2 "" H 2300 2750 50  0001 C CNN
+F 3 "" H 2300 2750 50  0001 C CNN
+	1    2300 2750
 	1    0    0    -1
 $EndComp
 Wire Wire Line
-	2850 2750 2850 2700
+	2300 2750 2300 2700
+$Comp
+L C_Small C21
+U 1 1 631185E3
+P 3050 2200
+F 0 "C21" V 3300 2150 50  0000 L CNN
+F 1 "1nF" V 3200 2050 50  0000 L CNN
+F 2 "LCSDR:C_1206_0603" H 3050 2200 50  0001 C CNN
+F 3 "" H 3050 2200 50  0001 C CNN
+	1    3050 2200
+	0    -1   -1   0
+$EndComp
 Wire Wire Line
-	3000 2500 3100 2500
+	3150 2200 3600 2200
 Wire Wire Line
-	3100 2500 3100 2200
-Connection ~ 3100 2200
+	2950 2200 2500 2200
+Wire Wire Line
+	2450 2500 2750 2500
+Wire Wire Line
+	2750 2500 2750 2200
+Connection ~ 2750 2200
 $EndSCHEMATC

Commit message: add text to HPF/LPF sch
Parts:
- C21, C49: value 1nF -> 680pF
- C45, C47: value 360pF -> 270pF
- L13, L17: value 1uH -> 900nH
- L15: value 680nH -> 800nH
Other:
- note added: "40M (7Mhz) High Pass Filter"
Changed lines of the file:
@@
 P 3700 2200
 F 0 "C45" V 3950 2150 50  0000 L CNN
-F 1 "360pF" V 3850 2050 50  0000 L CNN
+F 1 "270pF" V 3850 2050 50  0000 L CNN
 F 2 "LCSDR:C_1206_0603" H 3700 2200 50  0001 C CNN
 F 3 "" H 3700 2200 50  0001 C CNN
@@
 P 4550 2200
 F 0 "C47" V 4800 2150 50  0000 L CNN
-F 1 "360pF" V 4700 2050 50  0000 L CNN
+F 1 "270pF" V 4700 2050 50  0000 L CNN
 F 2 "LCSDR:C_1206_0603" H 4550 2200 50  0001 C CNN
 F 3 "" H 4550 2200 50  0001 C CNN
@@
 P 5300 2200
 F 0 "C49" V 5550 2150 50  0000 L CNN
-F 1 "1nF" V 5450 2050 50  0000 L CNN
+F 1 "680pF" V 5450 2050 50  0000 L CNN
 F 2 "LCSDR:C_1206_0603" H 5300 2200 50  0001 C CNN
 F 3 "" H 5300 2200 50  0001 C CNN
@@
 P 4950 2400
 F 0 "L17" H 4980 2440 50  0000 L CNN
-F 1 "1uH" H 4980 2360 50  0000 L CNN
+F 1 "900nH" H 4980 2360 50  0000 L CNN
 F 2 "Choke_Toroid_ThroughHole:Choke_Toroid_6,5x13mm_Vertical" H 4950 2400 50  0001 C CNN
 F 3 "" H 4950 2400 50  0001 C CNN
@@
 P 4150 2400
 F 0 "L15" H 4180 2440 50  0000 L CNN
-F 1 "680nH" H 4180 2360 50  0000 L CNN
+F 1 "800nH" H 4180 2360 50  0000 L CNN
 F 2 "Choke_Toroid_ThroughHole:Choke_Toroid_6,5x13mm_Vertical" H 4150 2400 50  0001 C CNN
 F 3 "" H 4150 2400 50  0001 C CNN
@@
 P 3350 2400
 F 0 "L13" H 3380 2440 50  0000 L CNN
-F 1 "1uH" H 3380 2360 50  0000 L CNN
+F 1 "900nH" H 3380 2360 50  0000 L CNN
 F 2 "Choke_Toroid_ThroughHole:Choke_Toroid_6,5x13mm_Vertical" H 3350 2400 50  0001 C CNN
 F 3 "" H 3350 2400 50  0001 C CNN
@@
 $EndComp
 $Comp
-L GND #PWR121
+L GND #PWR0117
 U 1 1 630A3972
 P 4950 2600
-F 0 "#PWR121" H 4950 2350 50  0001 C CNN
+F 0 "#PWR0117" H 4950 2350 50  0001 C CNN
 F 1 "GND" H 4950 2450 50  0000 C CNN
 F 2 "" H 4950 2600 50  0001 C CNN
@@
 $EndComp
 $Comp
-L GND #PWR120
+L GND #PWR0118
 U 1 1 630A39B4
 P 4150 2600
-F 0 "#PWR120" H 4150 2350 50  0001 C CNN
+F 0 "#PWR0118" H 4150 2350 50  0001 C CNN
 F 1 "GND" H 4150 2450 50  0000 C CNN
 F 2 "" H 4150 2600 50  0001 C CNN
@@
 $EndComp
 $Comp
-L GND #PWR119
+L GND #PWR0119
 U 1 1 630A39EF
 P 3350 2600
-F 0 "#PWR119" H 3350 2350 50  0001 C CNN
+F 0 "#PWR0119" H 3350 2350 50  0001 C CNN
 F 1 "GND" H 3350 2450 50  0000 C CNN
 F 2 "" H 3350 2600 50  0001 C CNN
@@
 $EndComp
 $Comp
-L GND #PWR122
+L GND #PWR0120
 U 1 1 630C7FC1
 P 6250 2750
-F 0 "#PWR122" H 6250 2500 50  0001 C CNN
+F 0 "#PWR0120" H 6250 2500 50  0001 C CNN
 F 1 "GND" H 6250 2600 50  0001 C CNN
 F 2 "" H 6250 2750 50  0001 C CNN
@@
 $EndComp
 $Comp
-L GND #PWR118
+L GND #PWR0121
 U 1 1 630C80FB
 P 2300 2750
-F 0 "#PWR118" H 2300 2500 50  0001 C CNN
+F 0 "#PWR0121" H 2300 2500 50  0001 C CNN
 F 1 "GND" H 2300 2600 50  0001 C CNN
 F 2 "" H 2300 2750 50  0001 C CNN
@@
 P 3050 2200
 F 0 "C21" V 3300 2150 50  0000 L CNN
-F 1 "1nF" V 3200 2050 50  0000 L CNN
+F 1 "680pF" V 3200 2050 50  0000 L CNN
 F 2 "LCSDR:C_1206_0603" H 3050 2200 50  0001 C CNN
 F 3 "" H 3050 2200 50  0001 C CNN
@@
 	2750 2500 2750 2200
 Connection ~ 2750 2200
+Text Notes 3250 1700 0    60   ~ 0
+ 40M  (7Mhz) High Pass Filter
 $EndSCHEMATC
