File: PCBs_OpA/RX998.sch (KiCad schematic (older format))
At the start: 26 parts, among them J1 MIC, Q7 BF998, U7 NE5532

Commit message: operational amplifier Direct detection receiver
Parts:
- removed C23: 10nF, LCSDR:C_1206_0603, symbol C_Small
- added Q? (x4): BF998, TO_SOT_Packages_SMD:SOT-143, symbol BF998
Connections:
- wire segments 60 -> 61
Other:
- moved on the sheet: C14, C16, C22, C24, C3, C4, C5, C54, C6, C7, J1, Q7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

Commit message: add LPF/HPF RFSimm models
Parts:
- removed C54: 100nF, LCSDR:C_1206_0603, symbol C_Small
- removed R27: 910, LCSDR:R_1206_0603, symbol R_Small
- removed U7: NE5532, Housings_SOIC:SOIC-8_3.9x4.9mm_Pitch1.27mm, symbol NE5532
- added C23, C39: 56pF, LCSDR:C_1206_0603, symbol C_Small
- added C37, C40, C42, C43: 100nF, LCSDR:C_1206_0603, symbol C_Small
- added C41: 10uF, Capacitors_THT:CP_Radial_D5.0mm_P2.00mm, symbol CP_Small
- added L3: 100uH, Choke_Axial_ThroughHole:Choke_Horizontal_RM10mm, symbol L_Small
- added L4: 100mH, Choke_Toroid_ThroughHole:Choke_Toroid_8x16mm_Vertical, symbol L_Small
- added Q12: BF998, TO_SOT_Packages_SMD:SOT-143, symbol BF998
- added R16: 10K, LCSDR:R_1206_0603, symbol R_Small
- added T1, T2: Transformer_1_4, LCSDR:TF14, symbol Transformer_1_4
- added Y3, Y4, Y5, Y6, Y7, Y8, Y9: Crystal, Crystals:Crystal_HC49-U_Vertical, symbol Crystal
- C14, C7: value 27nF -> 10nF
- C16: value 1uF -> 56pF
- C24: value 10nF -> 100nF
- C3: value 100nF -> 10nF
- C5: value 33nF -> 100nF
- C6: value 33nF -> 56pF
- R10: value 910 -> 1.5K
- R2: value 2K -> 220
- R22: value 2.7K -> 100
- R23: value 1.2K -> 10K
- R24: value 2K -> 300
- R25: value 910 -> 100
- R26: value 5.1K -> 220
- gave numbers to parts that had none: 4
Connections:
- net labels added: CLK2
- wire segments 61 -> 104
Other:
- moved on the sheet: C14, C22, C24, C4, C7, J1, Q10, Q11, Q3, Q5, Q7, R5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

Commit message: release gerber files
Parts:
- added J17: QER, Pin_Headers:Pin_Header_Straight_1x01_Pitch2.54mm, symbol Conn_01x01
Connections:
- net GND: now also J17.1 (Pin_1)
Changed lines of the file:
@@
 $EndComp
 $Comp
-L +12V #PWR052
+L +12V #PWR74
 U 1 1 6305C3FB
 P 9500 1750
-F 0 "#PWR052" H 9500 1600 50  0001 C CNN
+F 0 "#PWR74" H 9500 1600 50  0001 C CNN
 F 1 "+12V" H 9500 1900 50  0000 C CNN
 F 2 "" H 9500 1750 50  0001 C CNN
@@
 $EndComp
 $Comp
-L GND #PWR053
+L GND #PWR65
 U 1 1 6305C92E
 P 8200 4550
-F 0 "#PWR053" H 8200 4300 50  0001 C CNN
+F 0 "#PWR65" H 8200 4300 50  0001 C CNN
 F 1 "GND" H 8200 4400 50  0001 C CNN
 F 2 "" H 8200 4550 50  0001 C CNN
@@
 $EndComp
 $Comp
-L GND #PWR054
+L GND #PWR71
 U 1 1 6305CDF4
 P 9050 5500
-F 0 "#PWR054" H 9050 5250 50  0001 C CNN
+F 0 "#PWR71" H 9050 5250 50  0001 C CNN
 F 1 "GND" H 9050 5350 50  0001 C CNN
 F 2 "" H 9050 5500 50  0001 C CNN
@@
 $EndComp
 $Comp
-L GND #PWR055
+L GND #PWR73
 U 1 1 6305D55E
 P 9450 5500
-F 0 "#PWR055" H 9450 5250 50  0001 C CNN
+F 0 "#PWR73" H 9450 5250 50  0001 C CNN
 F 1 "GND" H 9450 5350 50  0001 C CNN
 F 2 "" H 9450 5500 50  0001 C CNN
@@
 $EndComp
 $Comp
-L GND #PWR056
+L GND #PWR67
 U 1 1 6305D895
 P 8600 5400
-F 0 "#PWR056" H 8600 5150 50  0001 C CNN
+F 0 "#PWR67" H 8600 5150 50  0001 C CNN
 F 1 "GND" H 8600 5250 50  0001 C CNN
 F 2 "" H 8600 5400 50  0001 C CNN
@@
 $EndComp
 $Comp
-L GND #PWR057
+L GND #PWR59
 U 1 1 6309F154
 P 6350 4900
-F 0 "#PWR057" H 6350 4650 50  0001 C CNN
+F 0 "#PWR59" H 6350 4650 50  0001 C CNN
 F 1 "GND" H 6350 4750 50  0001 C CNN
 F 2 "" H 6350 4900 50  0001 C CNN
@@
 $EndComp
 $Comp
-L GND #PWR058
+L GND #PWR55
 U 1 1 630E31E5
 P 4000 5300
-F 0 "#PWR058" H 4000 5050 50  0001 C CNN
+F 0 "#PWR55" H 4000 5050 50  0001 C CNN
 F 1 "GND" H 4000 5150 50  0001 C CNN
 F 2 "" H 4000 5300 50  0001 C CNN
@@
 $EndComp
 $Comp
-L +12V #PWR059
+L +12V #PWR56
 U 1 1 630E3241
 P 4850 1950
-F 0 "#PWR059" H 4850 1800 50  0001 C CNN
+F 0 "#PWR56" H 4850 1800 50  0001 C CNN
 F 1 "+12V" V 4850 2200 50  0000 C CNN
 F 2 "" H 4850 1950 50  0001 C CNN
@@
 $EndComp
 $Comp
-L GND #PWR060
+L GND #PWR54
 U 1 1 6311B006
 P 3250 4300
-F 0 "#PWR060" H 3250 4050 50  0001 C CNN
+F 0 "#PWR54" H 3250 4050 50  0001 C CNN
 F 1 "GND" H 3250 4150 50  0001 C CNN
 F 2 "" H 3250 4300 50  0001 C CNN
@@
 $EndComp
 $Comp
-L GND #PWR061
+L GND #PWR53
 U 1 1 631277DF
 P 2350 2350
-F 0 "#PWR061" H 2350 2100 50  0001 C CNN
+F 0 "#PWR53" H 2350 2100 50  0001 C CNN
 F 1 "GND" H 2350 2200 50  0001 C CNN
 F 2 "" H 2350 2350 50  0001 C CNN
@@
 $EndComp
 $Comp
-L GND #PWR062
+L GND #PWR57
 U 1 1 6312B80F
 P 5600 3500
-F 0 "#PWR062" H 5600 3250 50  0001 C CNN
+F 0 "#PWR57" H 5600 3250 50  0001 C CNN
 F 1 "GND" H 5600 3350 50  0001 C CNN
 F 2 "" H 5600 3500 50  0001 C CNN
@@
 $EndComp
 $Comp
-L GND #PWR063
+L GND #PWR58
 U 1 1 6312BBE8
 P 6300 3500
-F 0 "#PWR063" H 6300 3250 50  0001 C CNN
+F 0 "#PWR58" H 6300 3250 50  0001 C CNN
 F 1 "GND" H 6300 3350 50  0001 C CNN
 F 2 "" H 6300 3500 50  0001 C CNN
@@
 $EndComp
 $Comp
-L GND #PWR064
+L GND #PWR61
 U 1 1 6312C996
 P 7000 3500
-F 0 "#PWR064" H 7000 3250 50  0001 C CNN
+F 0 "#PWR61" H 7000 3250 50  0001 C CNN
 F 1 "GND" H 7000 3350 50  0001 C CNN
 F 2 "" H 7000 3500 50  0001 C CNN
@@
 $EndComp
 $Comp
-L GND #PWR065
+L GND #PWR63
 U 1 1 6312CB80
 P 7750 3500
-F 0 "#PWR065" H 7750 3250 50  0001 C CNN
+F 0 "#PWR63" H 7750 3250 50  0001 C CNN
 F 1 "GND" H 7750 3350 50  0001 C CNN
 F 2 "" H 7750 3500 50  0001 C CNN
@@
 $EndComp
 $Comp
-L GND #PWR066
+L GND #PWR70
 U 1 1 6312DAF0
 P 9000 3500
-F 0 "#PWR066" H 9000 3250 50  0001 C CNN
+F 0 "#PWR70" H 9000 3250 50  0001 C CNN
 F 1 "GND" H 9000 3350 50  0001 C CNN
 F 2 "" H 9000 3500 50  0001 C CNN
@@
 $EndComp
 $Comp
-L GND #PWR067
+L GND #PWR69
 U 1 1 6312EE5D
 P 8800 2150
-F 0 "#PWR067" H 8800 1900 50  0001 C CNN
+F 0 "#PWR69" H 8800 1900 50  0001 C CNN
 F 1 "GND" H 8800 2000 50  0001 C CNN
 F 2 "" H 8800 2150 50  0001 C CNN
@@
 $EndComp
 $Comp
-L GND #PWR068
+L GND #PWR72
 U 1 1 63130293
 P 9450 3900
-F 0 "#PWR068" H 9450 3650 50  0001 C CNN
+F 0 "#PWR72" H 9450 3650 50  0001 C CNN
 F 1 "GND" H 9450 3750 50  0001 C CNN
 F 2 "" H 9450 3900 50  0001 C CNN
@@
 $EndComp
 $Comp
-L GND #PWR069
+L GND #PWR75
 U 1 1 63130494
 P 9800 3900
-F 0 "#PWR069" H 9800 3650 50  0001 C CNN
+F 0 "#PWR75" H 9800 3650 50  0001 C CNN
 F 1 "GND" H 9800 3750 50  0001 C CNN
 F 2 "" H 9800 3900 50  0001 C CNN
@@
 $EndComp
 $Comp
-L GND #PWR070
+L GND #PWR76
 U 1 1 63130D16
 P 10200 2150
-F 0 "#PWR070" H 10200 1900 50  0001 C CNN
+F 0 "#PWR76" H 10200 1900 50  0001 C CNN
 F 1 "GND" H 10200 2000 50  0001 C CNN
 F 2 "" H 10200 2150 50  0001 C CNN
@@
 CLK2
 $Comp
-L +12V #PWR071
+L +12V #PWR66
 U 1 1 63134981
 P 8600 4250
-F 0 "#PWR071" H 8600 4100 50  0001 C CNN
+F 0 "#PWR66" H 8600 4100 50  0001 C CNN
 F 1 "+12V" H 8600 4400 50  0000 C CNN
 F 2 "" H 8600 4250 50  0001 C CNN
@@
 $EndComp
 $Comp
-L GND #PWR072
+L GND #PWR64
 U 1 1 631351E0
 P 7900 5300
-F 0 "#PWR072" H 7900 5050 50  0001 C CNN
+F 0 "#PWR64" H 7900 5050 50  0001 C CNN
 F 1 "GND" H 7900 5150 50  0001 C CNN
 F 2 "" H 7900 5300 50  0001 C CNN
@@
 $EndComp
 $Comp
-L GND #PWR073
+L GND #PWR62
 U 1 1 63135B39
 P 7250 5300
-F 0 "#PWR073" H 7250 5050 50  0001 C CNN
+F 0 "#PWR62" H 7250 5050 50  0001 C CNN
 F 1 "GND" H 7250 5150 50  0001 C CNN
 F 2 "" H 7250 5300 50  0001 C CNN
@@
 Connection ~ 7250 4850
 $Comp
-L GND #PWR074
+L GND #PWR68
 U 1 1 63143AF7
 P 8700 3500
-F 0 "#PWR074" H 8700 3250 50  0001 C CNN
+F 0 "#PWR68" H 8700 3250 50  0001 C CNN
 F 1 "GND" H 8700 3350 50  0001 C CNN
 F 2 "" H 8700 3500 50  0001 C CNN
@@
 Connection ~ 8500 2950
 Connection ~ 9000 2950
+$Comp
+L Conn_01x01 J17
+U 1 1 6326EA8A
+P 6750 2100
+F 0 "J17" H 6750 2200 50  0000 C CNN
+F 1 "QER" H 6750 2000 50  0000 C CNN
+F 2 "Pin_Headers:Pin_Header_Straight_1x01_Pitch2.54mm" H 6750 2100 50  0001 C CNN
+F 3 "" H 6750 2100 50  0001 C CNN
+	1    6750 2100
+	1    0    0    -1
+$EndComp
+$Comp
+L GND #PWR60
+U 1 1 6326EA91
+P 6500 2100
+F 0 "#PWR60" H 6500 1850 50  0001 C CNN
+F 1 "GND" H 6500 1950 50  0001 C CNN
+F 2 "" H 6500 2100 50  0001 C CNN
+F 3 "" H 6500 2100 50  0001 C CNN
+	1    6500 2100
+	0    1    1    0
+$EndComp
+Wire Wire Line
+	6500 2100 6550 2100
 $EndSCHEMATC
