File: PCBs/PowerSupplay.sch (KiCad schematic (older format))
At the start: 11 parts, among them J8 Jack-DC, U4 LM1117-5.0, U5 LM1117-3.3

Commit message: discret, simple, CH340E
Parts:
- removed U4: LM1117-5.0, TO_SOT_Packages_SMD:SOT-223-3_TabPin2, symbol LM1117-5.0
- added U3: L78L05_TO92, TO_SOT_Packages_THT:TO-92_Inline_Narrow_Oval, symbol L78L05_TO92
Connections:
- net +12V: now also U5.3 (VI), U3.3 (VI)
- net +5V: now also U3.1 (VO); no longer U5.3 (VI)
- net GND: now also U3.2 (GND)
Changed lines of the file:
@@
 LIBS:BF998
 LIBS:relays
+LIBS:stm32
+LIBS:Interface_USB
+LIBS:Arduino
 LIBS:LCSDR-cache
 EELAYER 25 0
@@
 $EndDescr
 $Comp
-L LM1117-5.0 U4
-U 1 1 6253C1F5
-P 4600 1250
-F 0 "U4" H 4450 1500 50  0000 C CNN
-F 1 "LM1117-5.0" H 4400 1400 50  0000 L CNN
-F 2 "TO_SOT_Packages_SMD:SOT-223-3_TabPin2" H 4600 1250 50  0001 C CNN
-F 3 "" H 4600 1250 50  0001 C CNN
-	1    4600 1250
-	1    0    0    -1
-$EndComp
-$Comp
 L LM1117-3.3 U5
 U 1 1 6253C1FC
@@
 $EndComp
 $Comp
-L GND #PWR25
+L GND #PWR016
 U 1 1 6253C203
 P 4600 1550
-F 0 "#PWR25" H 4600 1300 50  0001 C CNN
+F 0 "#PWR016" H 4600 1300 50  0001 C CNN
 F 1 "GND" H 4600 1400 50  0001 C CNN
 F 2 "" H 4600 1550 50  0001 C CNN
@@
 $EndComp
 $Comp
-L GND #PWR28
+L GND #PWR017
 U 1 1 6253C210
 P 5050 1550
-F 0 "#PWR28" H 5050 1300 50  0001 C CNN
+F 0 "#PWR017" H 5050 1300 50  0001 C CNN
 F 1 "GND" H 5050 1400 50  0001 C CNN
 F 2 "" H 5050 1550 50  0001 C CNN
@@
 $EndComp
 $Comp
-L GND #PWR29
+L GND #PWR018
 U 1 1 6253C216
 P 5550 1550
-F 0 "#PWR29" H 5550 1300 50  0001 C CNN
+F 0 "#PWR018" H 5550 1300 50  0001 C CNN
 F 1 "GND" H 5550 1400 50  0001 C CNN
 F 2 "" H 5550 1550 50  0001 C CNN
@@
 $EndComp
 $Comp
-L +5V #PWR30
+L +5V #PWR019
 U 1 1 6253C223
 P 5600 1250
-F 0 "#PWR30" H 5600 1100 50  0001 C CNN
+F 0 "#PWR019" H 5600 1100 50  0001 C CNN
 F 1 "+5V" V 5600 1450 50  0000 C CNN
 F 2 "" H 5600 1250 50  0001 C CNN
@@
 $EndComp
 $Comp
-L GND #PWR21
+L GND #PWR020
 U 1 1 6253C230
 P 3450 1550
-F 0 "#PWR21" H 3450 1300 50  0001 C CNN
+F 0 "#PWR020" H 3450 1300 50  0001 C CNN
 F 1 "GND" H 3450 1400 50  0001 C CNN
 F 2 "" H 3450 1550 50  0001 C CNN
@@
 $EndComp
 $Comp
-L GND #PWR22
+L GND #PWR021
 U 1 1 6253C236
 P 3950 1550
-F 0 "#PWR22" H 3950 1300 50  0001 C CNN
+F 0 "#PWR021" H 3950 1300 50  0001 C CNN
 F 1 "GND" H 3950 1400 50  0001 C CNN
 F 2 "" H 3950 1550 50  0001 C CNN
@@
 $EndComp
 $Comp
-L GND #PWR23
+L GND #PWR022
 U 1 1 6253C24A
 P 3950 3800
-F 0 "#PWR23" H 3950 3550 50  0001 C CNN
+F 0 "#PWR022" H 3950 3550 50  0001 C CNN
 F 1 "GND" H 3950 3650 50  0001 C CNN
 F 2 "" H 3950 3800 50  0001 C CNN
@@
 $EndComp
 $Comp
-L GND #PWR24
+L GND #PWR023
 U 1 1 6253C257
 P 4400 3800
-F 0 "#PWR24" H 4400 3550 50  0001 C CNN
+F 0 "#PWR023" H 4400 3550 50  0001 C CNN
 F 1 "GND" H 4400 3650 50  0001 C CNN
 F 2 "" H 4400 3800 50  0001 C CNN
@@
 $EndComp
 $Comp
-L GND #PWR26
+L GND #PWR024
 U 1 1 6253C25D
 P 4900 3800
-F 0 "#PWR26" H 4900 3550 50  0001 C CNN
+F 0 "#PWR024" H 4900 3550 50  0001 C CNN
 F 1 "GND" H 4900 3650 50  0001 C CNN
 F 2 "" H 4900 3800 50  0001 C CNN
@@
 $EndComp
 $Comp
-L +3.3V #PWR27
+L +3.3V #PWR025
 U 1 1 6253C26A
 P 5000 3500
-F 0 "#PWR27" H 5000 3350 50  0001 C CNN
+F 0 "#PWR025" H 5000 3350 50  0001 C CNN
 F 1 "+3.3V" V 5000 3750 50  0000 C CNN
 F 2 "" H 5000 3500 50  0001 C CNN
@@
 $EndComp
 $Comp
-L +5V #PWR20
-U 1 1 6253C270
-P 3200 3500
-F 0 "#PWR20" H 3200 3350 50  0001 C CNN
-F 1 "+5V" V 3200 3700 50  0000 C CNN
-F 2 "" H 3200 3500 50  0001 C CNN
-F 3 "" H 3200 3500 50  0001 C CNN
-	1    3200 3500
-	0    -1   -1   0
-$EndComp
-$Comp
-L GND #PWR16
+L GND #PWR026
 U 1 1 6253C290
 P 1700 1950
-F 0 "#PWR16" H 1700 1700 50  0001 C CNN
+F 0 "#PWR026" H 1700 1700 50  0001 C CNN
 F 1 "GND" H 1700 1800 50  0001 C CNN
 F 2 "" H 1700 1950 50  0001 C CNN
@@
 $EndComp
 $Comp
-L +12V #PWR19
+L +12V #PWR027
 U 1 1 630B53DA
 P 2900 1100
-F 0 "#PWR19" H 2900 950 50  0001 C CNN
+F 0 "#PWR027" H 2900 950 50  0001 C CNN
 F 1 "+12V" H 2900 1240 50  0000 C CNN
 F 2 "" H 2900 1100 50  0001 C CNN
@@
 	4900 1250 5600 1250
 $Comp
-L +12VA #PWR18
+L +12VA #PWR028
 U 1 1 630BADB5
 P 2650 1600
-F 0 "#PWR18" H 2650 1450 50  0001 C CNN
+F 0 "#PWR028" H 2650 1450 50  0001 C CNN
 F 1 "+12VA" H 2650 1740 50  0000 C CNN
 F 2 "" H 2650 1600 50  0001 C CNN
@@
 $EndComp
 $Comp
-L GND #PWR17
+L GND #PWR029
 U 1 1 630BB4AD
 P 2200 2000
-F 0 "#PWR17" H 2200 1750 50  0001 C CNN
+F 0 "#PWR029" H 2200 1750 50  0001 C CNN
 F 1 "GND" H 2200 1850 50  0001 C CNN
 F 2 "" H 2200 2000 50  0001 C CNN
@@
 	2200 1800 2200 1700
 Connection ~ 2200 1700
+$Comp
+L +12V #PWR030
+U 1 1 63810041
+P 3200 3500
+F 0 "#PWR030" H 3200 3350 50  0001 C CNN
+F 1 "+12V" V 3200 3700 50  0000 C CNN
+F 2 "" H 3200 3500 50  0001 C CNN
+F 3 "" H 3200 3500 50  0001 C CNN
+	1    3200 3500
+	0    -1   -1   0
+$EndComp
+$Comp
+L L78L05_TO92 U3
+U 1 1 638101C3
+P 4600 1250
+F 0 "U3" H 4500 1500 50  0000 C CNN
+F 1 "L78L05_TO92" H 4500 1400 50  0000 L CNN
+F 2 "TO_SOT_Packages_THT:TO-92_Inline_Narrow_Oval" H 4600 1475 50  0001 C CIN
+F 3 "" H 4600 1200 50  0001 C CNN
+	1    4600 1250
+	1    0    0    -1
+$EndComp
 $EndSCHEMATC

Commit message: INIT project, si5351 generate properly frequency
Parts:
- removed C10: 100uF, Capacitors_THT:CP_Radial_D6.3mm_P2.50mm, symbol CP_Small
- removed C12: 100nF, LCSDR:C_1206_0603, symbol C_Small
- removed U3: L78L05_TO92, TO_SOT_Packages_THT:TO-92_Inline_Narrow_Oval, symbol L78L05_TO92
- C13, C9: footprint LCSDR:C_1206_0603 -> Capacitors_SMD:C_0603_HandSoldering
Changed lines of the file:
@@
 $Descr A4 11693 8268
 encoding utf-8
-Sheet 3 8
+Sheet 3 7
 Title ""
 Date ""
@@
 $EndComp
 $Comp
-L GND #PWR016
-U 1 1 6253C203
-P 4600 1550
-F 0 "#PWR016" H 4600 1300 50  0001 C CNN
-F 1 "GND" H 4600 1400 50  0001 C CNN
-F 2 "" H 4600 1550 50  0001 C CNN
-F 3 "" H 4600 1550 50  0001 C CNN
-	1    4600 1550
-	1    0    0    -1
-$EndComp
-$Comp
-L CP_Small C10
-U 1 1 6253C209
-P 5050 1450
-F 0 "C10" H 5150 1500 50  0000 L CNN
-F 1 "100uF" H 5150 1400 50  0000 L CNN
-F 2 "Capacitors_THT:CP_Radial_D6.3mm_P2.50mm" H 5050 1450 50  0001 C CNN
-F 3 "" H 5050 1450 50  0001 C CNN
-	1    5050 1450
-	1    0    0    -1
-$EndComp
-$Comp
-L GND #PWR017
-U 1 1 6253C210
-P 5050 1550
-F 0 "#PWR017" H 5050 1300 50  0001 C CNN
-F 1 "GND" H 5050 1400 50  0001 C CNN
-F 2 "" H 5050 1550 50  0001 C CNN
-F 3 "" H 5050 1550 50  0001 C CNN
-	1    5050 1550
-	1    0    0    -1
-$EndComp
-$Comp
-L GND #PWR018
-U 1 1 6253C216
-P 5550 1550
-F 0 "#PWR018" H 5550 1300 50  0001 C CNN
-F 1 "GND" H 5550 1400 50  0001 C CNN
-F 2 "" H 5550 1550 50  0001 C CNN
-F 3 "" H 5550 1550 50  0001 C CNN
-	1    5550 1550
-	1    0    0    -1
-$EndComp
-$Comp
-L C_Small C12
-U 1 1 6253C21C
-P 5550 1450
-F 0 "C12" H 5650 1500 50  0000 L CNN
-F 1 "100nF" H 5650 1400 50  0000 L CNN
-F 2 "LCSDR:C_1206_0603" H 5550 1450 50  0001 C CNN
-F 3 "" H 5550 1450 50  0001 C CNN
-	1    5550 1450
-	1    0    0    -1
-$EndComp
-$Comp
-L +5V #PWR019
-U 1 1 6253C223
-P 5600 1250
-F 0 "#PWR019" H 5600 1100 50  0001 C CNN
-F 1 "+5V" V 5600 1450 50  0000 C CNN
-F 2 "" H 5600 1250 50  0001 C CNN
-F 3 "" H 5600 1250 50  0001 C CNN
-	1    5600 1250
-	0    1    1    0
-$EndComp
-$Comp
 L CP_Small C8
 U 1 1 6253C229
@@
 $EndComp
 $Comp
-L GND #PWR020
+L GND #PWR014
 U 1 1 6253C230
 P 3450 1550
-F 0 "#PWR020" H 3450 1300 50  0001 C CNN
+F 0 "#PWR014" H 3450 1300 50  0001 C CNN
 F 1 "GND" H 3450 1400 50  0001 C CNN
 F 2 "" H 3450 1550 50  0001 C CNN
@@
 $EndComp
 $Comp
-L GND #PWR021
+L GND #PWR015
 U 1 1 6253C236
 P 3950 1550
-F 0 "#PWR021" H 3950 1300 50  0001 C CNN
+F 0 "#PWR015" H 3950 1300 50  0001 C CNN
 F 1 "GND" H 3950 1400 50  0001 C CNN
 F 2 "" H 3950 1550 50  0001 C CNN
@@
 F 0 "C9" H 4050 1500 50  0000 L CNN
 F 1 "100nF" H 4050 1400 50  0000 L CNN
-F 2 "LCSDR:C_1206_0603" H 3950 1450 50  0001 C CNN
+F 2 "Capacitors_SMD:C_0603_HandSoldering" H 3950 1450 50  0001 C CNN
 F 3 "" H 3950 1450 50  0001 C CNN
 	1    3950 1450
@@
 $EndComp
 $Comp
-L GND #PWR022
+L GND #PWR016
 U 1 1 6253C24A
 P 3950 3800
-F 0 "#PWR022" H 3950 3550 50  0001 C CNN
+F 0 "#PWR016" H 3950 3550 50  0001 C CNN
 F 1 "GND" H 3950 3650 50  0001 C CNN
 F 2 "" H 3950 3800 50  0001 C CNN
@@
 $EndComp
 $Comp
-L GND #PWR023
+L GND #PWR017
 U 1 1 6253C257
 P 4400 3800
-F 0 "#PWR023" H 4400 3550 50  0001 C CNN
+F 0 "#PWR017" H 4400 3550 50  0001 C CNN
 F 1 "GND" H 4400 3650 50  0001 C CNN
 F 2 "" H 4400 3800 50  0001 C CNN
@@
 $EndComp
 $Comp
-L GND #PWR024
+L GND #PWR018
 U 1 1 6253C25D
 P 4900 3800
-F 0 "#PWR024" H 4900 3550 50  0001 C CNN
+F 0 "#PWR018" H 4900 3550 50  0001 C CNN
 F 1 "GND" H 4900 3650 50  0001 C CNN
 F 2 "" H 4900 3800 50  0001 C CNN
@@
 F 0 "C13" H 5000 3750 50  0000 L CNN
 F 1 "100nF" H 5000 3650 50  0000 L CNN
-F 2 "LCSDR:C_1206_0603" H 4900 3700 50  0001 C CNN
+F 2 "Capacitors_SMD:C_0603_HandSoldering" H 4900 3700 50  0001 C CNN
 F 3 "" H 4900 3700 50  0001 C CNN
 	1    4900 3700
@@
 $EndComp
 $Comp
-L +3.3V #PWR025
+L +3.3V #PWR019
 U 1 1 6253C26A
 P 5000 3500
-F 0 "#PWR025" H 5000 3350 50  0001 C CNN
+F 0 "#PWR019" H 5000 3350 50  0001 C CNN
 F 1 "+3.3V" V 5000 3750 50  0000 C CNN
 F 2 "" H 5000 3500 50  0001 C CNN
@@
 $EndComp
 $Comp
-L GND #PWR026
+L GND #PWR020
 U 1 1 6253C290
 P 1700 1950
-F 0 "#PWR026" H 1700 1700 50  0001 C CNN
+F 0 "#PWR020" H 1700 1700 50  0001 C CNN
 F 1 "GND" H 1700 1800 50  0001 C CNN
 F 2 "" H 1700 1950 50  0001 C CNN
@@
 $EndComp
 $Comp
-L +12V #PWR027
+L +12V #PWR021
 U 1 1 630B53DA
-P 2900 1100
-F 0 "#PWR027" H 2900 950 50  0001 C CNN
-F 1 "+12V" H 2900 1240 50  0000 C CNN
-F 2 "" H 2900 1100 50  0001 C CNN
-F 3 "" H 2900 1100 50  0001 C CNN
-	1    2900 1100
-	1    0    0    -1
+P 3550 3500
+F 0 "#PWR021" H 3550 3350 50  0001 C CNN
+F 1 "+12V" V 3550 3750 50  0000 C CNN
+F 2 "" H 3550 3500 50  0001 C CNN
+F 3 "" H 3550 3500 50  0001 C CNN
+	1    3550 3500
+	0    -1   -1   0
 $EndComp
 Connection ~ 2900 1250
@@
 Wire Wire Line
 	1650 1700 2900 1700
-Wire Wire Line
-	3200 3500 3650 3500
 Connection ~ 4900 3500
 Connection ~ 4400 3500
@@
 Wire Wire Line
 	3450 1350 3450 1250
-Connection ~ 3950 1250
 Wire Wire Line
 	3950 1250 3950 1350
 Wire Wire Line
-	2900 1250 4300 1250
-Wire Wire Line
 	2900 1100 2900 1350
-Connection ~ 5550 1250
-Connection ~ 5050 1250
-Wire Wire Line
-	5550 1250 5550 1350
-Wire Wire Line
-	5050 1250 5050 1350
-Wire Wire Line
-	4900 1250 5600 1250
-$Comp
-L +12VA #PWR028
+$Comp
+L +12VA #PWR022
 U 1 1 630BADB5
 P 2650 1600
-F 0 "#PWR028" H 2650 1450 50  0001 C CNN
+F 0 "#PWR022" H 2650 1450 50  0001 C CNN
 F 1 "+12VA" H 2650 1740 50  0000 C CNN
 F 2 "" H 2650 1600 50  0001 C CNN
@@
 $EndComp
 $Comp
-L GND #PWR029
+L GND #PWR023
 U 1 1 630BB4AD
 P 2200 2000
-F 0 "#PWR029" H 2200 1750 50  0001 C CNN
+F 0 "#PWR023" H 2200 1750 50  0001 C CNN
 F 1 "GND" H 2200 1850 50  0001 C CNN
 F 2 "" H 2200 2000 50  0001 C CNN
@@
 	2200 1800 2200 1700
 Connection ~ 2200 1700
-$Comp
-L +12V #PWR030
-U 1 1 63810041
-P 3200 3500
-F 0 "#PWR030" H 3200 3350 50  0001 C CNN
-F 1 "+12V" V 3200 3700 50  0000 C CNN
-F 2 "" H 3200 3500 50  0001 C CNN
-F 3 "" H 3200 3500 50  0001 C CNN
-	1    3200 3500
-	0    -1   -1   0
-$EndComp
-$Comp
-L L78L05_TO92 U3
-U 1 1 638101C3
-P 4600 1250
-F 0 "U3" H 4500 1500 50  0000 C CNN
-F 1 "L78L05_TO92" H 4500 1400 50  0000 L CNN
-F 2 "TO_SOT_Packages_THT:TO-92_Inline_Narrow_Oval" H 4600 1475 50  0001 C CIN
-F 3 "" H 4600 1200 50  0001 C CNN
-	1    4600 1250
-	1    0    0    -1
-$EndComp
+Wire Wire Line
+	3950 1250 2900 1250
+Wire Wire Line
+	3550 3500 3650 3500
+$Comp
+L +12V #PWR024
+U 1 1 638424E1
+P 2900 1100
+F 0 "#PWR024" H 2900 950 50  0001 C CNN
+F 1 "+12V" H 2900 1250 50  0000 C CNN
+F 2 "" H 2900 1100 50  0001 C CNN
+F 3 "" H 2900 1100 50  0001 C CNN
+	1    2900 1100
+	1    0    0    -1
+$EndComp

Commit message: add printout, finish PCB, add LM7805
Parts:
- added U3: L7805, TO_SOT_Packages_THT:TO-220-3_Vertical, symbol L7805
Connections:
- net +12V: now also U3.1 (IN); no longer U5.3 (VI)
- net GND: now also U3.2 (GND)
- new net +5V: U3.3 (OUT), U5.3 (VI)
Changed lines of the file:
@@
 $EndComp
 $Comp
-L GND #PWR014
+L GND #PWR18
 U 1 1 6253C230
 P 3450 1550
-F 0 "#PWR014" H 3450 1300 50  0001 C CNN
+F 0 "#PWR18" H 3450 1300 50  0001 C CNN
 F 1 "GND" H 3450 1400 50  0001 C CNN
 F 2 "" H 3450 1550 50  0001 C CNN
@@
 $EndComp
 $Comp
-L GND #PWR015
+L GND #PWR21
 U 1 1 6253C236
 P 3950 1550
-F 0 "#PWR015" H 3950 1300 50  0001 C CNN
+F 0 "#PWR21" H 3950 1300 50  0001 C CNN
 F 1 "GND" H 3950 1400 50  0001 C CNN
 F 2 "" H 3950 1550 50  0001 C CNN
@@
 $EndComp
 $Comp
-L GND #PWR016
+L GND #PWR23
 U 1 1 6253C24A
 P 3950 3800
-F 0 "#PWR016" H 3950 3550 50  0001 C CNN
+F 0 "#PWR23" H 3950 3550 50  0001 C CNN
 F 1 "GND" H 3950 3650 50  0001 C CNN
 F 2 "" H 3950 3800 50  0001 C CNN
@@
 $EndComp
 $Comp
-L GND #PWR017
+L GND #PWR24
 U 1 1 6253C257
 P 4400 3800
-F 0 "#PWR017" H 4400 3550 50  0001 C CNN
+F 0 "#PWR24" H 4400 3550 50  0001 C CNN
 F 1 "GND" H 4400 3650 50  0001 C CNN
 F 2 "" H 4400 3800 50  0001 C CNN
@@
 $EndComp
 $Comp
-L GND #PWR018
+L GND #PWR26
 U 1 1 6253C25D
 P 4900 3800
-F 0 "#PWR018" H 4900 3550 50  0001 C CNN
+F 0 "#PWR26" H 4900 3550 50  0001 C CNN
 F 1 "GND" H 4900 3650 50  0001 C CNN
 F 2 "" H 4900 3800 50  0001 C CNN
@@
 $EndComp
 $Comp
-L +3.3V #PWR019
+L +3.3V #PWR27
 U 1 1 6253C26A
 P 5000 3500
-F 0 "#PWR019" H 5000 3350 50  0001 C CNN
+F 0 "#PWR27" H 5000 3350 50  0001 C CNN
 F 1 "+3.3V" V 5000 3750 50  0000 C CNN
 F 2 "" H 5000 3500 50  0001 C CNN
@@
 $EndComp
 $Comp
-L GND #PWR020
+L GND #PWR14
 U 1 1 6253C290
 P 1700 1950
-F 0 "#PWR020" H 1700 1700 50  0001 C CNN
+F 0 "#PWR14" H 1700 1700 50  0001 C CNN
 F 1 "GND" H 1700 1800 50  0001 C CNN
 F 2 "" H 1700 1950 50  0001 C CNN
@@
 	1    0    0    -1
 $EndComp
-$Comp
-L +12V #PWR021
-U 1 1 630B53DA
-P 3550 3500
-F 0 "#PWR021" H 3550 3350 50  0001 C CNN
-F 1 "+12V" V 3550 3750 50  0000 C CNN
-F 2 "" H 3550 3500 50  0001 C CNN
-F 3 "" H 3550 3500 50  0001 C CNN
-	1    3550 3500
-	0    -1   -1   0
-$EndComp
 Connection ~ 2900 1250
 Wire Wire Line
@@
 	2900 1100 2900 1350
 $Comp
-L +12VA #PWR022
+L +12VA #PWR16
 U 1 1 630BADB5
 P 2650 1600
-F 0 "#PWR022" H 2650 1450 50  0001 C CNN
+F 0 "#PWR16" H 2650 1450 50  0001 C CNN
 F 1 "+12VA" H 2650 1740 50  0000 C CNN
 F 2 "" H 2650 1600 50  0001 C CNN
@@
 $EndComp
 $Comp
-L GND #PWR023
+L GND #PWR15
 U 1 1 630BB4AD
 P 2200 2000
-F 0 "#PWR023" H 2200 1750 50  0001 C CNN
+F 0 "#PWR15" H 2200 1750 50  0001 C CNN
 F 1 "GND" H 2200 1850 50  0001 C CNN
 F 2 "" H 2200 2000 50  0001 C CNN
@@
 Connection ~ 2200 1700
 Wire Wire Line
-	3950 1250 2900 1250
+	2900 1250 3950 1250
 Wire Wire Line
 	3550 3500 3650 3500
 $Comp
-L +12V #PWR024
+L +12V #PWR17
 U 1 1 638424E1
 P 2900 1100
-F 0 "#PWR024" H 2900 950 50  0001 C CNN
+F 0 "#PWR17" H 2900 950 50  0001 C CNN
 F 1 "+12V" H 2900 1250 50  0000 C CNN
 F 2 "" H 2900 1100 50  0001 C CNN
@@
 	1    0    0    -1
 $EndComp
+$Comp
+L L7805 U3
+U 1 1 639E7452
+P 3950 2400
+F 0 "U3" H 3800 2525 50  0000 C CNN
+F 1 "L7805" H 3950 2525 50  0000 L CNN
+F 2 "TO_SOT_Packages_THT:TO-220-3_Vertical" H 3975 2250 50  0001 L CIN
+F 3 "" H 3950 2350 50  0001 C CNN
+	1    3950 2400
+	1    0    0    -1
+$EndComp
+$Comp
+L +12V #PWR19
+U 1 1 639E751B
+P 3450 2400
+F 0 "#PWR19" H 3450 2250 50  0001 C CNN
+F 1 "+12V" V 3450 2650 50  0000 C CNN
+F 2 "" H 3450 2400 50  0001 C CNN
+F 3 "" H 3450 2400 50  0001 C CNN
+	1    3450 2400
+	0    -1   -1   0
+$EndComp
+Wire Wire Line
+	3450 2400 3650 2400
+$Comp
+L GND #PWR22
+U 1 1 639E7562
+P 3950 2700
+F 0 "#PWR22" H 3950 2450 50  0001 C CNN
+F 1 "GND" H 3950 2550 50  0001 C CNN
+F 2 "" H 3950 2700 50  0001 C CNN
+F 3 "" H 3950 2700 50  0001 C CNN
+	1    3950 2700
+	1    0    0    -1
+$EndComp
+Wire Wire Line
+	4250 2400 4650 2400
+$Comp
+L +5V #PWR25
+U 1 1 639E7652
+P 4650 2400
+F 0 "#PWR25" H 4650 2250 50  0001 C CNN
+F 1 "+5V" V 4650 2600 50  0000 C CNN
+F 2 "" H 4650 2400 50  0001 C CNN
+F 3 "" H 4650 2400 50  0001 C CNN
+	1    4650 2400
+	0    1    1    0
+$EndComp
+$Comp
+L +5V #PWR20
+U 1 1 639E76B5
+P 3550 3500
+F 0 "#PWR20" H 3550 3350 50  0001 C CNN
+F 1 "+5V" V 3550 3700 50  0000 C CNN
+F 2 "" H 3550 3500 50  0001 C CNN
+F 3 "" H 3550 3500 50  0001 C CNN
+	1    3550 3500
+	0    -1   -1   0
+$EndComp
 $EndSCHEMATC
