File: PCBs/RX.sch (KiCad schematic (older format))
At the start: 26 parts, among them J1 MIC, Q3 BFR93A, Q7 BF998

Commit message: INIT project, si5351 generate properly frequency
Parts:
- C3, C4, C5: footprint LCSDR:C_1206_0603 -> Capacitors_SMD:C_0603_HandSoldering
Changed lines of the file:
@@
 $Descr A4 11693 8268
 encoding utf-8
-Sheet 5 8
+Sheet 5 7
 Title ""
 Date ""
@@
 $EndComp
 $Comp
-L +12V #PWR051
+L +12V #PWR047
 U 1 1 6305C3FB
 P 4750 1400
-F 0 "#PWR051" H 4750 1250 50  0001 C CNN
+F 0 "#PWR047" H 4750 1250 50  0001 C CNN
 F 1 "+12V" V 4750 1600 50  0000 C CNN
 F 2 "" H 4750 1400 50  0001 C CNN
@@
 $EndComp
 $Comp
-L GND #PWR052
+L GND #PWR048
 U 1 1 6305C92E
 P 5200 1750
-F 0 "#PWR052" H 5200 1500 50  0001 C CNN
+F 0 "#PWR048" H 5200 1500 50  0001 C CNN
 F 1 "GND" H 5200 1600 50  0001 C CNN
 F 2 "" H 5200 1750 50  0001 C CNN
@@
 Connection ~ 6100 2300
 $Comp
-L GND #PWR053
+L GND #PWR049
 U 1 1 6305CDF4
 P 6100 2750
-F 0 "#PWR053" H 6100 2500 50  0001 C CNN
+F 0 "#PWR049" H 6100 2500 50  0001 C CNN
 F 1 "GND" H 6100 2600 50  0001 C CNN
 F 2 "" H 6100 2750 50  0001 C CNN
@@
 Connection ~ 6500 2400
 $Comp
-L GND #PWR054
+L GND #PWR050
 U 1 1 6305D55E
 P 6500 2750
-F 0 "#PWR054" H 6500 2500 50  0001 C CNN
+F 0 "#PWR050" H 6500 2500 50  0001 C CNN
 F 1 "GND" H 6500 2600 50  0001 C CNN
 F 2 "" H 6500 2750 50  0001 C CNN
@@
 	6500 2750 6500 2700
 $Comp
-L GND #PWR055
+L GND #PWR051
 U 1 1 6305D895
 P 5650 2650
-F 0 "#PWR055" H 5650 2400 50  0001 C CNN
+F 0 "#PWR051" H 5650 2400 50  0001 C CNN
 F 1 "GND" H 5650 2500 50  0001 C CNN
 F 2 "" H 5650 2650 50  0001 C CNN
@@
 Connection ~ 5000 2100
 $Comp
-L GND #PWR056
+L GND #PWR052
 U 1 1 6305E42E
 P 5000 2450
-F 0 "#PWR056" H 5000 2200 50  0001 C CNN
+F 0 "#PWR052" H 5000 2200 50  0001 C CNN
 F 1 "GND" H 5000 2300 50  0001 C CNN
 F 2 "" H 5000 2450 50  0001 C CNN
@@
 	4350 2100 4600 2100
 $Comp
-L GND #PWR057
+L GND #PWR053
 U 1 1 6305E6B0
 P 4450 2450
-F 0 "#PWR057" H 4450 2200 50  0001 C CNN
+F 0 "#PWR053" H 4450 2200 50  0001 C CNN
 F 1 "GND" H 4450 2300 50  0001 C CNN
 F 2 "" H 4450 2450 50  0001 C CNN
@@
 $EndComp
 $Comp
-L GND #PWR058
+L GND #PWR054
 U 1 1 6309F154
 P 3300 2250
-F 0 "#PWR058" H 3300 2000 50  0001 C CNN
+F 0 "#PWR054" H 3300 2000 50  0001 C CNN
 F 1 "GND" H 3300 2100 50  0001 C CNN
 F 2 "" H 3300 2250 50  0001 C CNN
@@
 $EndComp
 $Comp
-L GND #PWR059
+L GND #PWR055
 U 1 1 630BA840
 P 3800 2700
-F 0 "#PWR059" H 3800 2450 50  0001 C CNN
+F 0 "#PWR055" H 3800 2450 50  0001 C CNN
 F 1 "GND" H 3800 2550 50  0001 C CNN
 F 2 "" H 3800 2700 50  0001 C CNN
@@
 F 0 "C4" V 7800 3200 50  0000 L CNN
 F 1 "100nF" V 7700 3100 50  0000 L CNN
-F 2 "LCSDR:C_1206_0603" H 7550 3250 50  0001 C CNN
+F 2 "Capacitors_SMD:C_0603_HandSoldering" H 7550 3250 50  0001 C CNN
 F 3 "" H 7550 3250 50  0001 C CNN
 	1    7550 3250
@@
 	7200 3250 7200 3400
 $Comp
-L GND #PWR060
+L GND #PWR056
 U 1 1 63327041
 P 7200 3700
-F 0 "#PWR060" H 7200 3450 50  0001 C CNN
+F 0 "#PWR056" H 7200 3450 50  0001 C CNN
 F 1 "GND" H 7200 3550 50  0001 C CNN
 F 2 "" H 7200 3700 50  0001 C CNN
@@
 	7200 3700 7200 3600
 $Comp
-L GND #PWR061
+L GND #PWR057
 U 1 1 633270C2
 P 7950 3700
-F 0 "#PWR061" H 7950 3450 50  0001 C CNN
+F 0 "#PWR057" H 7950 3450 50  0001 C CNN
 F 1 "GND" H 7950 3550 50  0001 C CNN
 F 2 "" H 7950 3700 50  0001 C CNN
@@
 F 0 "C5" V 8650 2050 50  0000 L CNN
 F 1 "100nF" V 8550 1950 50  0000 L CNN
-F 2 "LCSDR:C_1206_0603" H 8400 2100 50  0001 C CNN
+F 2 "Capacitors_SMD:C_0603_HandSoldering" H 8400 2100 50  0001 C CNN
 F 3 "" H 8400 2100 50  0001 C CNN
 	1    8400 2100
@@
 	9600 2800 9800 2800
 $Comp
-L GND #PWR062
+L GND #PWR058
 U 1 1 633285BF
 P 8850 3350
-F 0 "#PWR062" H 8850 3100 50  0001 C CNN
+F 0 "#PWR058" H 8850 3100 50  0001 C CNN
 F 1 "GND" H 8850 3200 50  0001 C CNN
 F 2 "" H 8850 3350 50  0001 C CNN
@@
 $EndComp
 $Comp
-L +12V #PWR063
+L +12V #PWR059
 U 1 1 633287BE
 P 7000 1350
-F 0 "#PWR063" H 7000 1200 50  0001 C CNN
+F 0 "#PWR059" H 7000 1200 50  0001 C CNN
 F 1 "+12V" V 7000 1550 50  0000 C CNN
 F 2 "" H 7000 1350 50  0001 C CNN
@@
 F 0 "C3" H 7550 1600 50  0000 L CNN
 F 1 "100nF" H 7550 1500 50  0000 L CNN
-F 2 "LCSDR:C_1206_0603" H 7450 1550 50  0001 C CNN
+F 2 "Capacitors_SMD:C_0603_HandSoldering" H 7450 1550 50  0001 C CNN
 F 3 "" H 7450 1550 50  0001 C CNN
 	1    7450 1550
@@
 $EndComp
 $Comp
-L GND #PWR064
+L GND #PWR060
 U 1 1 633287CB
 P 7450 1700
-F 0 "#PWR064" H 7450 1450 50  0001 C CNN
+F 0 "#PWR060" H 7450 1450 50  0001 C CNN
 F 1 "GND" H 7450 1550 50  0001 C CNN
 F 2 "" H 7450 1700 50  0001 C CNN
