File: PCBs/SI5351.sch (KiCad schematic (older format))
At the start: 12 parts, among them J3 Calibration, Q1 2N7002, Q2 2N7002, U2 Si5351, Y1 25Mhz

Commit message: migrate to attiny1614
Parts:
- removed Q1, Q2: 2N7002, TO_SOT_Packages_SMD:SOT-23, symbol 2N7002
- removed R1, R3: 10K, Resistors_SMD:R_0603_HandSoldering, symbol R_Small
Connections:
- net SCL: now also R4.2, U2.4 (SCL)
- net SDA: now also R11.2, U2.5 (SDA)
- net CLK2: now reaches J3.1 (Pin_1), U2.6 (CLK2)
Changed lines of the file:
@@
 LIBS:Interface_USB
 LIBS:Arduino
+LIBS:MCU_Microchip_ATtiny
 LIBS:LCSDR-cache
 EELAYER 25 0
@@
 Comment4 ""
 $EndDescr
-Text GLabel 2900 5050 0    60   BiDi ~ 0
+Text GLabel 3700 5050 0    60   BiDi ~ 0
 SDA
-Text GLabel 2850 3350 0    60   Output ~ 0
+Text GLabel 3700 3350 0    60   Output ~ 0
 SCL
 $Comp
@@
 $EndComp
 $Comp
-L +3.3V #PWR8
+L +3.3V #PWR02
 U 1 1 62501FD9
 P 5000 2500
-F 0 "#PWR8" H 5000 2350 50  0001 C CNN
+F 0 "#PWR02" H 5000 2350 50  0001 C CNN
 F 1 "+3.3V" H 5000 2640 50  0000 C CNN
 F 2 "" H 5000 2500 50  0001 C CNN
@@
 $EndComp
 $Comp
-L GND #PWR12
+L GND #PWR03
 U 1 1 62501FDF
 P 6250 3600
-F 0 "#PWR12" H 6250 3350 50  0001 C CNN
+F 0 "#PWR03" H 6250 3350 50  0001 C CNN
 F 1 "GND" H 6250 3450 50  0001 C CNN
 F 2 "" H 6250 3600 50  0001 C CNN
@@
 $EndComp
 $Comp
-L +3.3V #PWR11
+L +3.3V #PWR04
 U 1 1 62501FE5
 P 6200 2100
-F 0 "#PWR11" H 6200 1950 50  0001 C CNN
+F 0 "#PWR04" H 6200 1950 50  0001 C CNN
 F 1 "+3.3V" H 6200 2240 50  0000 C CNN
 F 2 "" H 6200 2100 50  0001 C CNN
@@
 $EndComp
 $Comp
-L GND #PWR9
+L GND #PWR05
 U 1 1 6250203B
 P 5400 2700
-F 0 "#PWR9" H 5400 2450 50  0001 C CNN
+F 0 "#PWR05" H 5400 2450 50  0001 C CNN
 F 1 "GND" H 5400 2550 50  0001 C CNN
 F 2 "" H 5400 2700 50  0001 C CNN
@@
 	6450 3450 6450 3750
 Wire Wire Line
-	6450 3750 7400 3750
+	6450 3750 7600 3750
 Wire Wire Line
 	6550 3300 8000 3300
@@
 	4300 5050 4300 3450
 $Comp
-L +3.3V #PWR7
+L +3.3V #PWR06
 U 1 1 6250207D
 P 4000 4000
-F 0 "#PWR7" H 4000 3850 50  0001 C CNN
+F 0 "#PWR06" H 4000 3850 50  0001 C CNN
 F 1 "+3.3V" H 4000 4140 50  0000 C CNN
 F 2 "" H 4000 4000 50  0001 C CNN
@@
 $EndComp
 $Comp
-L GND #PWR10
+L GND #PWR07
 U 1 1 6253D2ED
 P 5800 2700
-F 0 "#PWR10" H 5800 2450 50  0001 C CNN
+F 0 "#PWR07" H 5800 2450 50  0001 C CNN
 F 1 "GND" H 5800 2550 50  0001 C CNN
 F 2 "" H 5800 2700 50  0001 C CNN
@@
 $EndComp
 $Comp
-L +3.3V #PWR6
+L +3.3V #PWR08
 U 1 1 630C0393
 P 4000 2150
-F 0 "#PWR6" H 4000 2000 50  0001 C CNN
+F 0 "#PWR08" H 4000 2000 50  0001 C CNN
 F 1 "+3.3V" H 4000 2290 50  0000 C CNN
 F 2 "" H 4000 2150 50  0001 C CNN
@@
 Connection ~ 4000 5050
 $Comp
-L GND #PWR13
+L GND #PWR09
 U 1 1 630C6EEC
 P 7800 4200
-F 0 "#PWR13" H 7800 3950 50  0001 C CNN
+F 0 "#PWR09" H 7800 3950 50  0001 C CNN
 F 1 "GND" H 7800 4050 50  0001 C CNN
 F 2 "" H 7800 4200 50  0001 C CNN
@@
 $EndComp
 Wire Wire Line
+	7800 4100 8050 4100
+Wire Wire Line
 	7800 4100 7800 4200
-$Comp
-L 2N7002 Q1
-U 1 1 63823E00
-P 3500 3250
-F 0 "Q1" V 3800 3300 50  0000 L CNN
-F 1 "2N7002" V 3900 3300 50  0000 L CNN
-F 2 "TO_SOT_Packages_SMD:SOT-23" H 3700 3175 50  0001 L CIN
-F 3 "" H 3500 3250 50  0001 L CNN
-	1    3500 3250
-	0    1    1    0
-$EndComp
-$Comp
-L +3.3V #PWR4
-U 1 1 63823F32
-P 3500 3000
-F 0 "#PWR4" H 3500 2850 50  0001 C CNN
-F 1 "+3.3V" H 3500 3140 50  0000 C CNN
-F 2 "" H 3500 3000 50  0001 C CNN
-F 3 "" H 3500 3000 50  0001 C CNN
-	1    3500 3000
-	1    0    0    -1
-$EndComp
-Wire Wire Line
-	3500 3000 3500 3050
-Wire Wire Line
-	2850 3350 3300 3350
-$Comp
-L R_Small R1
-U 1 1 63824069
-P 3150 2350
-F 0 "R1" H 3200 2400 50  0000 L CNN
-F 1 "10K" H 3200 2300 50  0000 L CNN
-F 2 "Resistors_SMD:R_0603_HandSoldering" H 3150 2350 50  0001 C CNN
-F 3 "" H 3150 2350 50  0001 C CNN
-	1    3150 2350
-	1    0    0    -1
-$EndComp
-Wire Wire Line
-	3150 2450 3150 3350
-Connection ~ 3150 3350
-Wire Wire Line
-	3150 2150 3150 2250
-$Comp
-L +5V #PWR2
-U 1 1 638241C8
-P 3150 2150
-F 0 "#PWR2" H 3150 2000 50  0001 C CNN
-F 1 "+5V" H 3150 2290 50  0000 C CNN
-F 2 "" H 3150 2150 50  0001 C CNN
-F 3 "" H 3150 2150 50  0001 C CNN
-	1    3150 2150
-	1    0    0    -1
-$EndComp
-$Comp
-L 2N7002 Q2
-U 1 1 638242E2
-P 3500 4950
-F 0 "Q2" V 3800 5000 50  0000 L CNN
-F 1 "2N7002" V 3900 5000 50  0000 L CNN
-F 2 "TO_SOT_Packages_SMD:SOT-23" H 3700 4875 50  0001 L CIN
-F 3 "" H 3500 4950 50  0001 L CNN
-	1    3500 4950
-	0    1    1    0
-$EndComp
-Wire Wire Line
-	2900 5050 3300 5050
-Connection ~ 3150 5050
-Wire Wire Line
-	3150 5050 3150 4300
-$Comp
-L R_Small R3
-U 1 1 638246FB
-P 3150 4200
-F 0 "R3" H 3200 4250 50  0000 L CNN
-F 1 "10K" H 3200 4150 50  0000 L CNN
-F 2 "Resistors_SMD:R_0603_HandSoldering" H 3150 4200 50  0001 C CNN
-F 3 "" H 3150 4200 50  0001 C CNN
-	1    3150 4200
-	1    0    0    -1
-$EndComp
-$Comp
-L +5V #PWR3
-U 1 1 6382473D
-P 3150 4000
-F 0 "#PWR3" H 3150 3850 50  0001 C CNN
-F 1 "+5V" H 3150 4140 50  0000 C CNN
-F 2 "" H 3150 4000 50  0001 C CNN
-F 3 "" H 3150 4000 50  0001 C CNN
-	1    3150 4000
-	1    0    0    -1
-$EndComp
-Wire Wire Line
-	3150 4000 3150 4100
-$Comp
-L +3.3V #PWR5
-U 1 1 638247BA
-P 3500 4650
-F 0 "#PWR5" H 3500 4500 50  0001 C CNN
-F 1 "+3.3V" H 3500 4790 50  0000 C CNN
-F 2 "" H 3500 4650 50  0001 C CNN
-F 3 "" H 3500 4650 50  0001 C CNN
-	1    3500 4650
-	1    0    0    -1
-$EndComp
-Wire Wire Line
-	3500 4650 3500 4750
 $Comp
 L Conn_01x02 J3
@@
 	1    0    0    -1
 $EndComp
-Wire Wire Line
-	7800 4100 8050 4100
+Text GLabel 7600 3750 2    60   Output ~ 0
+CLK2
+Connection ~ 7400 3750
 $EndSCHEMATC
